File: mic_tester/mic_tester.kicad_pcb (KiCad board)
At the start: 2 copper layers, 70 x 50 mm, 23 parts, among them J1 mic_connector, J2 amp_connector, J3 speaker_connector, J4 Power, U1 LM358, U2 LM386

Commit message: improve fix
Connections:
- R1 pad 1: Net-(R1-Pad1) -> Vcc
- R2 pad 2: Net-(R1-Pad1) -> Vcc
Routing:
- net Vcc: track 83.0 -> 106.8 mm
- net Net-(R1-Pad1): track 5.08 -> 0.00 mm
