File: mic_tester/mic_tester.kicad_sch (KiCad schematic)
At the start: 23 parts, among them J1 mic_connector, J2 amp_connector, J3 speaker_connector, J4 Power, U1 LM358, U2 LM386

Commit message: add text to schematics
Other:
- note added: "4V-12V"
Changed lines of the file:
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@@
+    (effects (font (size 1.27 1.27)) (justify left bottom))
+  )
+  (text "4V-12V" (at 44.45 21.59 0)
     (effects (font (size 1.27 1.27)) (justify left bottom))
   )

Commit message: fix error
Connections:
- net VCC: now also R1.1, R2.2
Changed lines of the file:
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@@
   (junction (at 110.49 104.14) (diameter 0) (color 0 0 0 0)
+  )
+  (junction (at 110.49 27.94) (diameter 0) (color 0 0 0 0)
   )
   (junction (at 125.73 53.34) (diameter 0) (color 0 0 0 0)
@@
     (stroke (width 0) (type default) (color 0 0 0 0))
   )
+  (wire (pts (xy 114.3 27.94) (xy 114.3 20.32))
+    (stroke (width 0) (type default) (color 0 0 0 0))
+  )
   (wire (pts (xy 148.59 40.64) (xy 154.94 40.64))
     (stroke (width 0) (type default) (color 0 0 0 0))
@@
     (stroke (width 0) (type default) (color 0 0 0 0))
   )
+  (wire (pts (xy 110.49 27.94) (xy 114.3 27.94))
+    (stroke (width 0) (type default) (color 0 0 0 0))
+  )
   (wire (pts (xy 77.47 43.18) (xy 90.17 43.18))
     (stroke (width 0) (type default) (color 0 0 0 0))
@@
     (stroke (width 0) (type default) (color 0 0 0 0))
   )
-  (wire (pts (xy 83.82 96.52) (xy 83.82 100.33))
+  (wire (pts (xy 83.82 96.52) (xy 83.82 124.46))
     (stroke (width 0) (type default) (color 0 0 0 0))
   )
@@
     (stroke (width 0) (type default) (color 0 0 0 0))
   )
-  (wire (pts (xy 88.9 100.33) (xy 83.82 100.33))
+  (wire (pts (xy 88.9 124.46) (xy 83.82 124.46))
     (stroke (width 0) (type default) (color 0 0 0 0))
   )
@@
     (effects (font (size 1.27 1.27)) (justify left))
     (property "Intersheet References" "${INTERSHEET_REFS}" (id 0) (at 148.5236 123.1106 0)
+      (effects (font (size 1.27 1.27)) (justify left) hide)
+    )
+  )
+  (global_label "Vcc" (shape input) (at 114.3 20.32 0) (fields_autoplaced)
+    (effects (font (size 1.27 1.27)) (justify left))
+    (property "Intersheet References" "${INTERSHEET_REFS}" (id 0) (at 119.9788 20.2406 0)
       (effects (font (size 1.27 1.27)) (justify left) hide)
     )
@@
     )
   )
-  (global_label "GND" (shape input) (at 88.9 100.33 0) (fields_autoplaced)
-    (effects (font (size 1.27 1.27)) (justify left))
-    (property "Intersheet References" "${INTERSHEET_REFS}" (id 0) (at 95.1836 100.2506 0)
-      (effects (font (size 1.27 1.27)) (justify left) hide)
-    )
+  (global_label "GND" (shape input) (at 88.9 124.46 0) (fields_autoplaced)
+    (effects (font (size 1.27 1.27)) (justify left))
+    (property "Intersheet References" "${INTERSHEET_REFS}" (id 0) (at 95.1836 124.3806 0)
+      (effects (font (size 1.27 1.27)) (justify left) hide)
+    )

Commit message: improve fix
Parts:
- RV1: footprint Potentiometer_THT:Potentiometer_Runtron_RM-065_Vertical -> Potentiometer_THT:Potentiometer_Piher_PT-6-V_Vertical
Changed lines of the file:
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@@
       (effects (font (size 1.27 1.27)) (justify right))
     )
-    (property "Footprint" "Potentiometer_THT:Potentiometer_Runtron_RM-065_Vertical" (id 2) (at 83.82 92.71 0)
+    (property "Footprint" "Potentiometer_THT:Potentiometer_Piher_PT-6-V_Vertical" (id 2) (at 83.82 92.71 0)
       (effects (font (size 1.27 1.27)) hide)
     )
@@
     )
     (path "/b59e0d69-36ca-4874-9a3b-18977012e6b1"
-      (reference "RV1") (unit 1) (value "10k") (footprint "Potentiometer_THT:Potentiometer_Runtron_RM-065_Vertical")
+      (reference "RV1") (unit 1) (value "10k") (footprint "Potentiometer_THT:Potentiometer_Piher_PT-6-V_Vertical")
     )
     (path "/4f41ede8-5aba-40d3-bb15-9886ab31ebe2"

Commit message: update to v1.1
Parts:
- C4, C8: footprint Capacitor_THT:CP_Radial_D10.0mm_P2.50mm -> Capacitor_THT:CP_Radial_D7.5mm_P2.50mm
Changed lines of the file:
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@@
   (junction (at 110.49 104.14) (diameter 0) (color 0 0 0 0)
   )
+  (junction (at 125.73 53.34) (diameter 0) (color 0 0 0 0)
+  )
+  (junction (at 170.18 43.18) (diameter 0) (color 0 0 0 0)
+  )
   (junction (at 110.49 27.94) (diameter 0) (color 0 0 0 0)
-  )
-  (junction (at 125.73 53.34) (diameter 0) (color 0 0 0 0)
-  )
-  (junction (at 170.18 43.18) (diameter 0) (color 0 0 0 0)
   )
   (junction (at 148.59 53.34) (diameter 0) (color 0 0 0 0)
@@
     (stroke (width 0) (type default) (color 0 0 0 0))
   )
-  (wire (pts (xy 114.3 27.94) (xy 114.3 20.32))
-    (stroke (width 0) (type default) (color 0 0 0 0))
-  )
   (wire (pts (xy 148.59 40.64) (xy 154.94 40.64))
     (stroke (width 0) (type default) (color 0 0 0 0))
@@
     (stroke (width 0) (type default) (color 0 0 0 0))
   )
-  (wire (pts (xy 110.49 27.94) (xy 114.3 27.94))
-    (stroke (width 0) (type default) (color 0 0 0 0))
-  )
   (wire (pts (xy 77.47 43.18) (xy 90.17 43.18))
     (stroke (width 0) (type default) (color 0 0 0 0))
@@
     (stroke (width 0) (type default) (color 0 0 0 0))
   )
+  (wire (pts (xy 110.49 20.32) (xy 110.49 27.94))
+    (stroke (width 0) (type default) (color 0 0 0 0))
+  )
   (polyline (pts (xy 246.38 69.85) (xy 283.21 69.85))
     (stroke (width 0) (type default) (color 0 0 0 0))
@@
   )
   (wire (pts (xy 80.01 83.82) (xy 83.82 83.82))
+    (stroke (width 0) (type default) (color 0 0 0 0))
+  )
+  (wire (pts (xy 114.3 20.32) (xy 110.49 20.32))
     (stroke (width 0) (type default) (color 0 0 0 0))
   )
@@
     (property "Reference" "C8" (id 0) (at 147.701 87.63 90))
     (property "Value" "220u" (id 1) (at 147.701 90.17 90))
-    (property "Footprint" "Capacitor_THT:CP_Radial_D10.0mm_P2.50mm" (id 2) (at 152.4 94.2848 0)
+    (property "Footprint" "Capacitor_THT:CP_Radial_D7.5mm_P2.50mm" (id 2) (at 152.4 94.2848 0)
       (effects (font (size 1.27 1.27)) hide)
     )
@@
       (effects (font (size 1.27 1.27)) hide)
     )
+    (pin "1")
+    (pin "2")
+    (pin "3")
     (pin "5")
     (pin "6")
     (pin "7")
+    (pin "4")
+    (pin "8")
   )
   (symbol (lib_id "Device:R") (at 105.41 43.18 90) (unit 1)
@@
     (property "Reference" "C4" (id 0) (at 175.641 35.56 90))
     (property "Value" "220u" (id 1) (at 175.641 38.1 90))
-    (property "Footprint" "Capacitor_THT:CP_Radial_D10.0mm_P2.50mm" (id 2) (at 180.34 42.2148 0)
+    (property "Footprint" "Capacitor_THT:CP_Radial_D7.5mm_P2.50mm" (id 2) (at 180.34 42.2148 0)
       (effects (font (size 1.27 1.27)) hide)
     )
@@
     (pin "2")
     (pin "3")
+    (pin "5")
+    (pin "6")
+    (pin "7")
+    (pin "4")
+    (pin "8")
   )
   (symbol (lib_id "Connector:Conn_01x02_Male") (at 168.91 97.79 180) (unit 1)
@@
       (effects (font (size 1.27 1.27)) hide)
     )
+    (pin "1")
+    (pin "2")
+    (pin "3")
+    (pin "5")
+    (pin "6")
+    (pin "7")
     (pin "4")
     (pin "8")
@@
     )
     (path "/42de3f85-8d22-4a91-ac22-6d7dab73449c"
-      (reference "C4") (unit 1) (value "220u") (footprint "Capacitor_THT:CP_Radial_D10.0mm_P2.50mm")
+      (reference "C4") (unit 1) (value "220u") (footprint "Capacitor_THT:CP_Radial_D7.5mm_P2.50mm")
     )
     (path "/fb24df25-1284-4e21-9a76-50321e8bc317"
@@
     )
     (path "/1ecaff67-dc68-4ef1-be1d-7b5e0356a4de"
-      (reference "C8") (unit 1) (value "220u") (footprint "Capacitor_THT:CP_Radial_D10.0mm_P2.50mm")
+      (reference "C8") (unit 1) (value "220u") (footprint "Capacitor_THT:CP_Radial_D7.5mm_P2.50mm")
     )
     (path "/321e2df7-ced6-4c62-b165-8193090f5c43"
